Commit message: done

File: body.urdf (robot description, URDF)
Before this commit: robot robot, 6 links, 5 joints
Links:
- added link Link10, mass 1; collision box size=0.4570785949956508 0.3782888991663589 0.47424198403872425; visual box size=0.4570785949956508 0.3782888991663589 0.47424198403872425
- added link Link7, mass 1; collision box size=0.3002513106870079 0.05929644354391289 0.14219435760050764; visual box size=0.3002513106870079 0.05929644354391289 0.14219435760050764
- added link Link8, mass 1; collision box size=0.17433466906818218 0.0369727476411183 0.21181720822114886; visual box size=0.17433466906818218 0.0369727476411183 0.21181720822114886
- added link Link9, mass 1; collision box size=0.19954699994093755 0.35667518558501093 0.3983115054907689; visual box size=0.19954699994093755 0.35667518558501093 0.3983115054907689
- link Link1: geometry collision box size=0.28238037309439223 0.36047816047590114 0.2935030490408063; visual box size=0.28238037309439223 0.36047816047590114 0.2935030490408063
- link Link2: geometry collision box size=0.025138879111411272 0.4255267181619639 0.01501976469306282; visual box size=0.025138879111411272 0.4255267181619639 0.01501976469306282
- link Link3: geometry collision box size=0.34918723469710095 0.4670382745413493 0.23493779371267182; visual box size=0.34918723469710095 0.4670382745413493 0.23493779371267182
- link Link4: geometry collision box size=0.17732732675038565 0.4573774499784223 0.060040481397707846; visual box size=0.17732732675038565 0.4573774499784223 0.060040481397707846
- link Link5: geometry collision box size=0.3473447877886872 0.40512516828825873 0.10359966163506729; visual box size=0.3473447877886872 0.40512516828825873 0.10359966163506729
- link Link6: geometry collision box size=0.22644400711938473 0.17351799234159332 0.46657208462569305; visual box size=0.22644400711938473 0.17351799234159332 0.46657208462569305
Joints:
- added joint Link6_Link7: type revolute, parent Link6, child Link7, origin xyz=0 0.0 0.0 rpy=0 0 0, axis 1 0 0, limit lower=-3.14159 upper=3.14159 effort=0.0 velocity=0.0
- added joint Link7_Link8: type revolute, parent Link7, child Link8, origin xyz=-0.15012565534350394 -0.029648221771956446 0.14219435760050764 rpy=0 0 0, axis 0 1 0, limit lower=-3.14159 upper=3.14159 effort=0.0 velocity=0.0
- added joint Link8_Link9: type revolute, parent Link8, child Link9, origin xyz=0.0 0 0.0 rpy=0 0 0, axis 0 1 0, limit lower=-3.14159 upper=3.14159 effort=0.0 velocity=0.0
- added joint Link9_Link10: type revolute, parent Link9, child Link10, origin xyz=0.19954699994093755 0 0.0 rpy=0 0 0, axis 0 1 0, limit lower=-3.14159 upper=3.14159 effort=0.0 velocity=0.0
- joint Link1_Link2: origin xyz=0.03304236523396262 0 0.3190513140909531 rpy=0 0 0 -> xyz=0.14119018654719612 0 1.2935030490408064 rpy=0 0 0
- joint Link2_Link3: axis 0 1 0 -> 1 0 0; origin xyz=0.42384011714147785 0 0.13592080034438836 rpy=0 0 0 -> xyz=0.012569439555705636 -0.21276335908098196 0.0 rpy=0 0 0
- joint Link3_Link4: axis 0 1 0 -> 1 0 0; origin xyz=0.18871405631231997 0 0.12759028221349816 rpy=0 0 0 -> xyz=0 0.0 0.0 rpy=0 0 0
- joint Link4_Link5: origin xyz=0.4558763822671102 0 0.29963039541311554 rpy=0 0 0 -> xyz=0.08866366337519282 0.22868872498921114 0.0 rpy=0 0 0
- joint Link5_Link6: axis 0 1 0 -> 1 0 0; origin xyz=0.07733837970252738 0 0.12972691509796813 rpy=0 0 0 -> xyz=0.1736723938943436 0.20256258414412937 0.10359966163506729 rpy=0 0 0
